File: 2024KASAboard/2024KASAboard.kicad_sch (KiCad schematic)
At the start: 2 parts, among them U1 Pico, U2 BME280

Commit message: add-i2c
Connections:
- net at U2.4 (SDI): now also U1.21 (GPIO16)
- net at U2.6 (SCK): now also U1.22 (GPIO17)
Changed lines of the file:
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@@
+	(wire
+		(pts
+			(xy 153.67 105.41) (xy 217.17 105.41)
+		)
+		(stroke
+			(width 0)
+			(type default)
+		)
+	)
+	(wire
+		(pts
+			(xy 217.17 105.41) (xy 217.17 78.74)
+		)
+		(stroke
+			(width 0)
+			(type default)
+		)
+	)
 	(wire
 		(pts
@@
 	(wire
 		(pts
+			(xy 153.67 107.95) (xy 212.09 107.95)
+		)
+		(stroke
+			(width 0)
+			(type default)
+		)
+	)
+	(wire
+		(pts
 			(xy 167.64 78.74) (xy 167.64 69.85)
 		)
 		(stroke
+			(width 0)
+			(type default)
+		)
+	)
+	(wire
+		(pts
+			(xy 212.09 107.95) (xy 212.09 78.74)
+		)
+		(stroke

Commit message: shirakawa
Connections:
- net at U2.3 (CSB): now also U1.24 (GPIO18)
Other:
- moved on the sheet: U1, U2
Changed lines of the file:
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@@
 	(wire
 		(pts
-			(xy 153.67 105.41) (xy 217.17 105.41)
-		)
-		(stroke
-			(width 0)
-			(type default)
-		)
-	)
-	(wire
-		(pts
-			(xy 217.17 105.41) (xy 217.17 78.74)
-		)
-		(stroke
-			(width 0)
-			(type default)
-		)
-	)
-	(wire
-		(pts
-			(xy 204.47 78.74) (xy 167.64 78.74)
-		)
-		(stroke
-			(width 0)
-			(type default)
-		)
-	)
-	(wire
-		(pts
-			(xy 167.64 69.85) (xy 153.67 69.85)
-		)
-		(stroke
-			(width 0)
-			(type default)
-		)
-	)
-	(wire
-		(pts
-			(xy 207.01 78.74) (xy 207.01 90.17)
-		)
-		(stroke
-			(width 0)
-			(type default)
-		)
-	)
-	(wire
-		(pts
-			(xy 153.67 107.95) (xy 212.09 107.95)
-		)
-		(stroke
-			(width 0)
-			(type default)
-		)
-	)
-	(wire
-		(pts
-			(xy 167.64 78.74) (xy 167.64 69.85)
-		)
-		(stroke
-			(width 0)
-			(type default)
-		)
-	)
-	(wire
-		(pts
-			(xy 212.09 107.95) (xy 212.09 78.74)
-		)
-		(stroke
-			(width 0)
-			(type default)
-		)
-	)
-	(wire
-		(pts
-			(xy 207.01 90.17) (xy 153.67 90.17)
+			(xy 115.57 105.41) (xy 179.07 105.41)
+		)
+		(stroke
+			(width 0)
+			(type default)
+		)
+	)
+	(wire
+		(pts
+			(xy 171.45 78.74) (xy 171.45 100.33)
+		)
+		(stroke
+			(width 0)
+			(type default)
+		)
+	)
+	(wire
+		(pts
+			(xy 179.07 105.41) (xy 179.07 78.74)
+		)
+		(stroke
+			(width 0)
+			(type default)
+		)
+	)
+	(wire
+		(pts
+			(xy 166.37 78.74) (xy 129.54 78.74)
+		)
+		(stroke
+			(width 0)
+			(type default)
+		)
+	)
+	(wire
+		(pts
+			(xy 129.54 69.85) (xy 115.57 69.85)
+		)
+		(stroke
+			(width 0)
+			(type default)
+		)
+	)
+	(wire
+		(pts
+			(xy 115.57 100.33) (xy 171.45 100.33)
+		)
+		(stroke
+			(width 0)
+			(type default)
+		)
+	)
+	(wire
+		(pts
+			(xy 168.91 78.74) (xy 168.91 90.17)
+		)
+		(stroke
+			(width 0)
+			(type default)
+		)
+	)
+	(wire
+		(pts
+			(xy 115.57 107.95) (xy 173.99 107.95)
+		)
+		(stroke
+			(width 0)
+			(type default)
+		)
+	)
+	(wire
+		(pts
+			(xy 129.54 78.74) (xy 129.54 69.85)
+		)
+		(stroke
+			(width 0)
+			(type default)
+		)
+	)
+	(wire
+		(pts
+			(xy 173.99 107.95) (xy 173.99 78.74)
+		)
+		(stroke
+			(width 0)
+			(type default)
+		)
+	)
+	(wire
+		(pts
+			(xy 168.91 90.17) (xy 115.57 90.17)
 		)
 		(stroke
@@
 	(symbol
 		(lib_id "0_kasa_lib-2024-:BME280")
-		(at 210.82 72.39 0)
+		(at 172.72 72.39 0)
 		(unit 1)
 		(exclude_from_sim no)
@@
 		(fields_autoplaced yes)
 		(property "Reference" "U2"
-			(at 219.71 74.9299 0)
+			(at 181.61 74.9299 0)
 			(effects
 				(font
@@
 		)
 		(property "Value" "BME280"
-			(at 219.71 77.4699 0)
+			(at 181.61 77.4699 0)
 			(effects
 				(font
@@
 		)
 		(property "Footprint" ""
-			(at 213.36 71.12 0)
+			(at 175.26 71.12 0)
 			(effects
 				(font
@@
 		)
 		(property "Datasheet" ""
-			(at 213.36 71.12 0)
+			(at 175.26 71.12 0)
 			(effects
 				(font
@@
 		)
 		(property "Description" ""
-			(at 210.82 72.39 0)
+			(at 172.72 72.39 0)
 			(effects
 				(font
@@
 	(symbol
 		(lib_id "MCU_RaspberryPi_and_Boards:Pico")
-		(at 135.89 83.82 0)
+		(at 97.79 83.82 0)
 		(unit 1)
 		(exclude_from_sim no)
@@
 		(fields_autoplaced yes)
 		(property "Reference" "U1"
-			(at 135.89 52.07 0)
+			(at 97.79 52.07 0)
 			(effects
 				(font
@@
 		)
 		(property "Value" "Pico"
-			(at 135.89 54.61 0)
+			(at 97.79 54.61 0)
 			(effects
 				(font
@@
 		)
 		(property "Footprint" "RPi_Pico:RPi_Pico_SMD_TH"
-			(at 135.89 83.82 90)
+			(at 97.79 83.82 90)
 			(effects
 				(font
@@
 		)
 		(property "Datasheet" ""
-			(at 135.89 83.82 0)
+			(at 97.79 83.82 0)
 			(effects
 				(font
@@
 		)
 		(property "Description" ""
-			(at 135.89 83.82 0)
-			(effects
-				(font
+			(at 97.79 83.82 0)
+			(effects
+				(font

Commit message: apple
Connections:
- net at U2.5 (SDO): now also U1.26 (GPIO20)
Changed lines of the file:
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@@
+	(wire
+		(pts
+			(xy 176.53 78.74) (xy 176.53 111.76)
+		)
+		(stroke
+			(width 0)
+			(type default)
+		)
+	)
+	(wire
+		(pts
+			(xy 129.54 111.76) (xy 176.53 111.76)
+		)
+		(stroke
+			(width 0)
+			(type default)
+		)
+	)
+	(wire
+		(pts
+			(xy 129.54 95.25) (xy 115.57 95.25)
+		)
+		(stroke
+			(width 0)
+			(type default)
+		)
+	)
 	(wire
 		(pts
@@
 		)
 		(stroke
+			(width 0)
+			(type default)
+		)
+	)
+	(wire
+		(pts
+			(xy 129.54 111.76) (xy 129.54 95.25)
+		)
+		(stroke

Commit message: banana
Connections:
- net at U1.1 (GPIO0): now also U1.32 (GPIO27_ADC1)
- net at U1.34 (GPIO28_ADC2): now also U1.40 (VBUS)
Changed lines of the file:
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@@
+	(wire
+		(pts
+			(xy 121.92 52.07) (xy 121.92 80.01)
+		)
+		(stroke
+			(width 0)
+			(type default)
+		)
+	)
 	(wire
 		(pts
@@
 	(wire
 		(pts
+			(xy 80.01 59.69) (xy 77.47 59.69)
+		)
+		(stroke
+			(width 0)
+			(type default)
+		)
+	)
+	(wire
+		(pts
 			(xy 115.57 100.33) (xy 171.45 100.33)
+		)
+		(stroke
+			(width 0)
+			(type default)
+		)
+	)
+	(wire
+		(pts
+			(xy 77.47 59.69) (xy 77.47 52.07)
 		)
 		(stroke
@@
 	(wire
 		(pts
+			(xy 121.92 80.01) (xy 115.57 80.01)
+		)
+		(stroke
+			(width 0)
+			(type default)
+		)
+	)
+	(wire
+		(pts
+			(xy 125.73 74.93) (xy 125.73 59.69)
+		)
+		(stroke
+			(width 0)
+			(type default)
+		)
+	)
+	(wire
+		(pts
+			(xy 115.57 74.93) (xy 125.73 74.93)
+		)
+		(stroke
+			(width 0)
+			(type default)
+		)
+	)
+	(wire
+		(pts
+			(xy 77.47 52.07) (xy 121.92 52.07)
+		)
+		(stroke
+			(width 0)
+			(type default)
+		)
+	)
+	(wire
+		(pts
 			(xy 129.54 111.76) (xy 129.54 95.25)
 		)
@@
 		)
 		(stroke
+			(width 0)
+			(type default)
+		)
+	)
+	(wire
+		(pts
+			(xy 125.73 59.69) (xy 115.57 59.69)
+		)
+		(stroke
